File: Thupp-Right/_autosave-Thupp-Right.kicad_pcb (KiCad board)
At the start: 2 copper layers, 43 parts, among them U1 nice_nano

Commit message: fully routed 1st attempt
Routing:
- net COL0: track 78.5 -> 132.2 mm
- net COL1: track 77.9 -> 109.0 mm
- net COL2: track 91.9 -> 99.3 mm
Changed lines of the file:
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@@
     (thickness 1.6)
     (drawings 232)
-    (tracks 186)
+    (tracks 196)
     (zones 0)
     (modules 43)
@@
   (segment (start 53.198391 99.773711) (end 53.198391 76.307555) (width 0.254) (layer B.Cu) (net 26))
   (segment (start 42.813354 110.158748) (end 53.198391 99.773711) (width 0.254) (layer B.Cu) (net 26))
+  (segment (start 90.531263 111.945622) (end 93.657994 108.818891) (width 0.254) (layer B.Cu) (net 26))
+  (segment (start 43.186015 111.945622) (end 90.531263 111.945622) (width 0.254) (layer B.Cu) (net 26))
+  (segment (start 42.813354 111.572961) (end 43.186015 111.945622) (width 0.254) (layer B.Cu) (net 26))
+  (segment (start 42.813354 110.158748) (end 42.813354 111.572961) (width 0.254) (layer B.Cu) (net 26))
   (segment (start 71.771907 54.211354) (end 72.771906 55.211353) (width 0.254) (layer B.Cu) (net 27))
   (segment (start 71.771907 37.418258) (end 71.771907 54.211354) (width 0.254) (layer B.Cu) (net 27))
@@
   (segment (start 62.887513 106.303345) (end 71.994905 97.195953) (width 0.254) (layer B.Cu) (net 27))
   (segment (start 62.887513 108.609518) (end 62.887513 106.303345) (width 0.254) (layer B.Cu) (net 27))
+  (segment (start 79.468309 105.566657) (end 65.930374 105.566657) (width 0.254) (layer B.Cu) (net 27))
+  (segment (start 65.930374 105.566657) (end 62.887513 108.609518) (width 0.254) (layer B.Cu) (net 27))
+  (segment (start 80.657851 106.756199) (end 79.468309 105.566657) (width 0.254) (layer B.Cu) (net 27))
+  (segment (start 92.1758 106.756199) (end 80.657851 106.756199) (width 0.254) (layer B.Cu) (net 27))
   (segment (start 90.566498 46.355242) (end 91.566497 45.355243) (width 0.254) (layer B.Cu) (net 28))
   (segment (start 90.566498 63.150264) (end 90.566498 46.355242) (width 0.254) (layer B.Cu) (net 28))
@@
   (segment (start 75.2475 96.025262) (end 82.088009 102.865771) (width 0.254) (layer B.Cu) (net 28))
   (segment (start 75.2475 76.269298) (end 75.2475 96.025262) (width 0.254) (layer B.Cu) (net 28))
+  (segment (start 86.304442 100.568122) (end 82.088009 104.784555) (width 0.254) (layer B.Cu) (net 28))
+  (segment (start 87.729216 100.568122) (end 86.304442 100.568122) (width 0.254) (layer B.Cu) (net 28))
   (segment (start 109.363014 50.557947) (end 110.363013 51.557946) (width 0.254) (layer B.Cu) (net 29))
   (segment (start 109.363014 33.762922) (end 109.363014 50.557947) (width 0.254) (layer B.Cu) (net 29))

Commit message: fully routed 1st attempt
Routing:
- net ROW3: track 46.1 -> 61.1 mm
- net COL1: track 109.0 -> 108.0 mm
Changed lines of the file:
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@@
     (thickness 1.6)
     (drawings 232)
-    (tracks 196)
+    (tracks 197)
     (zones 0)
     (modules 43)
@@
   (segment (start 69.810176 100.584) (end 71.57536 102.349184) (width 0.254) (layer F.Cu) (net 23))
   (segment (start 57.960544 100.584) (end 69.810176 100.584) (width 0.254) (layer F.Cu) (net 23))
+  (segment (start 79.624162 98.038516) (end 83.282632 94.380046) (width 0.254) (layer F.Cu) (net 23))
+  (segment (start 75.886028 98.038516) (end 79.624162 98.038516) (width 0.254) (layer F.Cu) (net 23))
+  (segment (start 71.57536 102.349184) (end 75.886028 98.038516) (width 0.254) (layer F.Cu) (net 23))
   (segment (start 58.122361 109.16) (end 53.77 109.16) (width 0.25) (layer F.Cu) (net 24))
   (segment (start 62.677668 104.604693) (end 58.122361 109.16) (width 0.25) (layer F.Cu) (net 24))
@@
   (segment (start 62.887513 106.303345) (end 71.994905 97.195953) (width 0.254) (layer B.Cu) (net 27))
   (segment (start 62.887513 108.609518) (end 62.887513 106.303345) (width 0.254) (layer B.Cu) (net 27))
-  (segment (start 79.468309 105.566657) (end 65.930374 105.566657) (width 0.254) (layer B.Cu) (net 27))
-  (segment (start 65.930374 105.566657) (end 62.887513 108.609518) (width 0.254) (layer B.Cu) (net 27))
-  (segment (start 80.657851 106.756199) (end 79.468309 105.566657) (width 0.254) (layer B.Cu) (net 27))
-  (segment (start 92.1758 106.756199) (end 80.657851 106.756199) (width 0.254) (layer B.Cu) (net 27))
+  (segment (start 90.322481 108.609518) (end 92.1758 106.756199) (width 0.254) (layer B.Cu) (net 27))
+  (segment (start 62.887513 108.609518) (end 90.322481 108.609518) (width 0.254) (layer B.Cu) (net 27))
   (segment (start 90.566498 46.355242) (end 91.566497 45.355243) (width 0.254) (layer B.Cu) (net 28))
   (segment (start 90.566498 63.150264) (end 90.566498 46.355242) (width 0.254) (layer B.Cu) (net 28))
